Commit message: update yamaprox

File: fetch_gazebo/robots/sensor_links.xacro (robot description, xacro)
@@ -9,5 +9,5 @@
         </geometry>
         <material name="">
-          <color rgba="0 0.500 0 1"/>
+          <color rgba="0 0.500 0 0.1"/>
         </material>
       </visual>
@@ -43,5 +43,15 @@
     <xacro:arg name="sensor_name" default="proximity_sensor_tf/${l_r}/${frame}/${sensor_num}" />
     <!-- Define sensor link -->
-    <link name="proximity_sensor_tf/${l_r}/${frame}/${sensor_num}" />
+    <link name="proximity_sensor_tf/${l_r}/${frame}/${sensor_num}">
+        <visual>
+          <origin rpy="0 0 0" xyz="0.01 0.01 0"/>
+          <geometry>
+            <box size="0.005 0.005 0.005"/>
+          </geometry>
+          <material name="">
+            <color rgba="1.0 0 0 1"/>
+          </material>
+        </visual>
+    </link>
     <joint name="proximity_sensor_joint/${l_r}/${frame}/${sensor_num}" type="fixed">
       <parent link="gripper_link"/>
